Commit message: coorected wheel size
Signed-off-by: Tanishq Chaudhary <tanishqchaudhary101010@gmail.com>

File: robots_description/urdf/amr1.xacro (robot description, xacro)
@@ -3,11 +3,11 @@
   <xacro:include filename="$(find robots_description)/urdf/amr_base_common.xacro"/>
   <!-- customize AMR-1 -->
-  <xacro:property name="wheel_radius" value="0.08"/>
-  <xacro:property name="wheel_width"  value="0.05"/>
-  <xacro:property name="wheel_base"   value="0.45"/>
-  <xacro:property name="chassis_length" value="0.60"/>
-  <xacro:property name="chassis_width"  value="0.45"/>
-  <xacro:property name="chassis_height" value="0.20"/>
-  <xacro:property name="mass_chassis" value="15.0"/>
+  <xacro:property name="wheel_radius" value="0.05"/>
+  <xacro:property name="wheel_width"  value="0.025"/>
+  <xacro:property name="wheel_base"   value="0.4"/>
+  <xacro:property name="chassis_length" value="0.5"/>
+  <xacro:property name="chassis_width"  value="0.3"/>
+  <xacro:property name="chassis_height" value="0.10"/>
+  <xacro:property name="mass_chassis" value="100.0"/>
   <!-- base_link (chassis) -->
   <link name="base_link">
@@ -33,5 +33,5 @@
     <parent link="base_link"/>
     <child link="wheel_left"/>
-    <origin xyz="0 ${wheel_base/2} ${wheel_radius}" rpy="0 0 0"/>
+    <origin xyz="0 ${wheel_base/2} ${chassis_height/4}" rpy="0 0 0"/>
     <axis xyz="0 1 0"/>
   </joint>
@@ -39,5 +39,5 @@
     <parent link="base_link"/>
     <child link="wheel_right"/>
-    <origin xyz="0 ${-wheel_base/2} ${wheel_radius}" rpy="0 0 0"/>
+    <origin xyz="0 ${-wheel_base/2} ${chassis_height/4}" rpy="0 0 0"/>
     <axis xyz="0 1 0"/>
   </joint>

File: robots_description/urdf/amr2.xacro (robot description, xacro)
@@ -3,11 +3,11 @@
   <xacro:include filename="$(find robots_description)/urdf/amr_base_common.xacro"/>
   <!-- customize AMR-2 -->
-  <xacro:property name="wheel_radius" value="0.09"/>
-  <xacro:property name="wheel_width"  value="0.06"/>
-  <xacro:property name="wheel_base"   value="0.48"/>
-  <xacro:property name="chassis_length" value="0.70"/>
-  <xacro:property name="chassis_width"  value="0.55"/>
-  <xacro:property name="chassis_height" value="0.22"/>
-  <xacro:property name="mass_chassis" value="20.0"/>
+  <xacro:property name="wheel_radius" value="0.1"/>
+  <xacro:property name="wheel_width"  value="0.05"/>
+  <xacro:property name="wheel_base"   value=".75"/>
+  <xacro:property name="chassis_length" value="1.0"/>
+  <xacro:property name="chassis_width"  value="0.6"/>
+  <xacro:property name="chassis_height" value="0.2"/>
+  <xacro:property name="mass_chassis" value="200.0"/>
   <!-- base -->
   <link name="base_link">

File: robots_description/urdf/amr_base_common.xacro (robot description, xacro)
@@ -27,5 +27,5 @@
     <link name="${name}">
       <visual>
-        <origin xyz="0 0 0" rpy="0 0 0"/>
+        <origin xyz="0 0 0" rpy="1.57 0 0"/>
         <geometry>
           <cylinder radius="${radius}" length="${width}"/>
@@ -33,5 +33,5 @@
       </visual>
       <collision>
-        <origin xyz="0 0 0" rpy="0 0 0"/>
+        <origin xyz="0 0 0" rpy="1.57 0 0"/>
         <geometry>
           <cylinder radius="${radius}" length="${width}"/>
