Commit message: fix
Signed-off-by: Tanishq Chaudhary <tanishqchaudhary101010@gmail.com>

File: robots_description/urdf/amr2.xacro (robot description, xacro)
@@ -28,5 +28,5 @@
     <parent link="base_link"/>
     <child link="wheel_left"/>
-    <origin xyz="0 ${wheel_base/2} ${wheel_radius}" rpy="0 0 0"/>
+    <origin xyz="0 ${wheel_base/2} ${chassis_height/4}" rpy="0 0 0"/>
     <axis xyz="0 1 0"/>
   </joint>
@@ -34,5 +34,5 @@
     <parent link="base_link"/>
     <child link="wheel_right"/>
-    <origin xyz="0 ${-wheel_base/2} ${wheel_radius}" rpy="0 0 0"/>
+    <origin xyz="0 ${-wheel_base/2} ${chassis_height/4}" rpy="0 0 0"/>
     <axis xyz="0 1 0"/>
   </joint>
