Commit message: lint
Signed-off-by: Tanishq Chaudhary <tanishqchaudhary101010@gmail.com>

File: robots_description/urdf/tug.core.xacro (robot description, xacro)
@@ -1,4 +1,5 @@
 <?xml version="1.0"?>
-<robot name="tug" xmlns:xacro="http://www.ros.org/wiki/xacro">
+<robot name="tug"
+  xmlns:xacro="http://www.ros.org/wiki/xacro">
   <xacro:include filename="$(find robots_description)/urdf/tug.model.xacro"/>
   <xacro:arg name="robot_name" default="tug_X"/>

File: robots_description/urdf/tug.gazebo.xacro (robot description, xacro)
@@ -1,35 +1,68 @@
 <?xml version="1.0"?>
-<robot name="tug_gazebo" xmlns:xacro="http://ros.org/wiki/xacro">
-  <xacro:arg name="robot_name" default="tug_X"/>
-  <xacro:macro name="tug_gazebo" params="robot_name">
-  <xacro:property name="base_length" value="0.6"/>
-  <xacro:property name="base_width"  value="0.45"/>
-  <xacro:property name="base_height" value="0.18"/>
-  <xacro:property name="wheel_radius" value="0.08"/>
-  <xacro:property name="wheel_width" value="0.04"/>
-  <xacro:property name="wheel_gap_from_base" value="0.01"/>
-  <xacro:property name="wheel_separation" value="${base_width/2 + wheel_width/2 + wheel_gap_from_base}"/>
-  <gazebo>
-		<plugin name='${robot_name}_diff_drive_gazebo_plugin' filename='libgazebo_ros_diff_drive.so'>
-			<ros>
-			  <namespace>${robot_name}</namespace>
-			</ros>
-			<!-- wheels -->
-			<left_joint>${robot_name}/joint_left_wheel</left_joint>
-			<right_joint>${robot_name}/joint_right_wheel</right_joint>
-			<!-- kinematics -->
-			<wheel_separation>${wheel_separation}</wheel_separation>
-			<wheel_diameter>${2*wheel_radius}</wheel_diameter>
-			<!-- limits -->
-			<max_wheel_torque>20</max_wheel_torque>
-			<max_wheel_acceleration>1.0</max_wheel_acceleration>
-			<!-- output -->
-			<publish_odom>true</publish_odom>
-			<publish_odom_tf>true</publish_odom_tf>
-			<publish_wheel_tf>true</publish_wheel_tf>
-			<odometry_frame>world</odometry_frame>
-			<robot_base_frame>${robot_name}/base_link</robot_base_frame>
-		</plugin>
-	</gazebo>
-	  </xacro:macro>
+<robot name="tug_gazebo"
+	xmlns:xacro="http://ros.org/wiki/xacro">
+	<xacro:arg name="robot_name" default="tug_X"/>
+	<xacro:macro name="tug_gazebo" params="robot_name">
+		<xacro:property name="base_length" value="0.6"/>
+		<xacro:property name="base_width" value="0.45"/>
+		<xacro:property name="base_height" value="0.18"/>
+		<xacro:property name="wheel_radius" value="0.08"/>
+		<xacro:property name="wheel_width" value="0.04"/>
+		<xacro:property name="wheel_gap_from_base" value="0.01"/>
+		<xacro:property name="wheel_separation" value="${base_width/2 + wheel_width/2 + wheel_gap_from_base}"/>
+		<gazebo reference="${robot_name}/left_wheel">
+			<mu1>1.0</mu1>
+			<mu2>1.0</mu2>
+			<kp>1000000.0</kp>
+			<kd>100.0</kd>
+			<minDepth>0.001</minDepth>
+			<maxVel>1.0</maxVel>
+		</gazebo>
+		<gazebo reference="${robot_name}/right_wheel">
+			<mu1>1.0</mu1>
+			<mu2>1.0</mu2>
+			<kp>1000000.0</kp>
+			<kd>100.0</kd>
+			<minDepth>0.001</minDepth>
+			<maxVel>1.0</maxVel>
+		</gazebo>
+		<gazebo reference="${robot_name}/caster_link_back">
+			<mu1>0.0</mu1>
+			<mu2>0.0</mu2>
+			<kp>1000000.0</kp>
+			<kd>100.0</kd>
+			<minDepth>0.001</minDepth>
+			<maxVel>1.0</maxVel>
+		</gazebo>
+		<gazebo reference="${robot_name}/caster_link_front">
+			<mu1>0.0</mu1>
+			<mu2>0.0</mu2>
+			<kp>1000000.0</kp>
+			<kd>100.0</kd>
+			<minDepth>0.001</minDepth>
+			<maxVel>1.0</maxVel>
+		</gazebo>
+		<gazebo>
+			<plugin name='${robot_name}_diff_drive_gazebo_plugin' filename='libgazebo_ros_diff_drive.so'>
+				<ros>
+					<namespace>${robot_name}</namespace>
+				</ros>
+				<!-- wheels -->
+				<left_joint>${robot_name}/joint_left_wheel</left_joint>
+				<right_joint>${robot_name}/joint_right_wheel</right_joint>
+				<!-- kinematics -->
+				<wheel_separation>${wheel_separation}</wheel_separation>
+				<wheel_diameter>${2*wheel_radius}</wheel_diameter>
+				<!-- limits -->
+				<max_wheel_torque>20</max_wheel_torque>
+				<max_wheel_acceleration>1.0</max_wheel_acceleration>
+				<!-- output -->
+				<publish_odom>true</publish_odom>
+				<publish_odom_tf>true</publish_odom_tf>
+				<publish_wheel_tf>true</publish_wheel_tf>
+				<odometry_frame>world</odometry_frame>
+				<robot_base_frame>${robot_name}/base_link</robot_base_frame>
+			</plugin>
+		</gazebo>
+	</xacro:macro>
 </robot>

File: robots_description/urdf/tug.model.xacro (robot description, xacro)
@@ -1,35 +1,36 @@
 <?xml version="1.0"?>
-<robot name="tug" xmlns:xacro="http://www.ros.org/wiki/xacro">
+<robot name="tug"
+  xmlns:xacro="http://www.ros.org/wiki/xacro">
   <xacro:arg name="robot_name" default="tug_X"/>
   <xacro:include filename="$(find robots_description)/urdf/tug.gazebo.xacro"/>
   <xacro:macro name="tug_model" params="robot_name">
-  <xacro:property name="base_length" value="0.6"/>
-  <xacro:property name="base_width"  value="0.45"/>
-  <xacro:property name="base_height" value="0.18"/>
-  <xacro:property name="wheel_radius" value="0.08"/>
-  <xacro:property name="wheel_width" value="0.04"/>
-  <xacro:property name="wheel_gap_from_base" value="0.01"/>
-  <xacro:property name="wheel_separation" value="${base_width/2 + wheel_width/2 + wheel_gap_from_base}"/>
+    <xacro:property name="base_length" value="0.6"/>
+    <xacro:property name="base_width" value="0.45"/>
+    <xacro:property name="base_height" value="0.18"/>
+    <xacro:property name="wheel_radius" value="0.08"/>
+    <xacro:property name="wheel_width" value="0.04"/>
+    <xacro:property name="wheel_gap_from_base" value="0.01"/>
+    <xacro:property name="wheel_separation" value="${base_width/2 + wheel_width/2 + wheel_gap_from_base}"/>
     <link name="${robot_name}/base_link">
-        <inertial>
-            <origin xyz="0 0 0" rpy="0 0 0"/>
-            <mass value="25.0"/>
-            <inertia ixx="1.0" ixy="0.0" ixz="0.0" iyy="1.2" iyz="0.0" izz="1.2"/>
-        </inertial>
-        <visual>
-            <geometry>
-                <box size="${base_length} ${base_width} ${base_height}"/>
-            </geometry>
-          <origin xyz="0 0 ${base_height/2}"/>
-          <material name="red">
-            <color rgba="1 0 0.01 1.0"/>
-          </material>
-        </visual>
-        <collision>
-          <geometry>
-            <box size="${base_length} ${base_width} ${base_height}"/>
-          </geometry>
-          <origin xyz="0 0 ${base_height/2}"/>
-        </collision>
+      <inertial>
+        <origin xyz="0 0 0" rpy="0 0 0"/>
+        <mass value="25.0"/>
+        <inertia ixx="1.0" ixy="0.0" ixz="0.0" iyy="1.2" iyz="0.0" izz="1.2"/>
+      </inertial>
+      <visual>
+        <geometry>
+          <box size="${base_length} ${base_width} ${base_height}"/>
+        </geometry>
+        <origin xyz="0 0 ${base_height/2}"/>
+        <material name="red">
+          <color rgba="1 0 0.01 1.0"/>
+        </material>
+      </visual>
+      <collision>
+        <geometry>
+          <box size="${base_length} ${base_width} ${base_height}"/>
+        </geometry>
+        <origin xyz="0 0 ${base_height/2}"/>
+      </collision>
     </link>
     <joint name="${robot_name}/joint_left_wheel" type="continuous">
@@ -40,125 +41,125 @@
     </joint>
     <link name="${robot_name}/left_wheel">
-        <inertial>
-            <origin xyz="0 0 0"/>
-            <mass value="0.8"/>
-            <inertia ixx="0.001" ixy="0.0" ixz="0.0" iyy="0.001" iyz="0.0" izz="0.002"/>
-        </inertial>
-        <visual>
-            <origin xyz="0 0 0" rpy="1.5708 0 0"/>
-            <geometry>
-                <cylinder radius="${wheel_radius}" length="${wheel_width}"/>
-            </geometry>
-            <material name="black">
-                <color rgba="0 0 0 1"/>
-            </material>
-        </visual>
-        <collision>
-            <origin xyz="0 0 0" rpy="1.5708 0 0"/>
-            <geometry>
-                <cylinder radius="${wheel_radius}" length="${wheel_width}"/>
-            </geometry>
-        </collision>
+      <inertial>
+        <origin xyz="0 0 0"/>
+        <mass value="0.8"/>
+        <inertia ixx="0.001" ixy="0.0" ixz="0.0" iyy="0.001" iyz="0.0" izz="0.002"/>
+      </inertial>
+      <visual>
+        <origin xyz="0 0 0" rpy="1.5708 0 0"/>
+        <geometry>
+          <cylinder radius="${wheel_radius}" length="${wheel_width}"/>
+        </geometry>
+        <material name="black">
+          <color rgba="0 0 0 1"/>
+        </material>
+      </visual>
+      <collision>
+        <origin xyz="0 0 0" rpy="1.5708 0 0"/>
+        <geometry>
+          <cylinder radius="${wheel_radius}" length="${wheel_width}"/>
+        </geometry>
+      </collision>
     </link>
     <joint name="${robot_name}/joint_right_wheel" type="continuous">
-        <parent link="${robot_name}/base_link"/>
-        <child link="${robot_name}/right_wheel"/>
-        <origin xyz="0 -${wheel_separation} ${wheel_radius/2}" rpy="0 0 0"/>
-        <axis xyz="0 1 0"/>
+      <parent link="${robot_name}/base_link"/>
+      <child link="${robot_name}/right_wheel"/>
+      <origin xyz="0 -${wheel_separation} ${wheel_radius/2}" rpy="0 0 0"/>
+      <axis xyz="0 1 0"/>
     </joint>
     <link name="${robot_name}/right_wheel">
-        <inertial>
-            <origin xyz="0 0 0"/>
-            <mass value="0.8"/>
-            <inertia ixx="0.001" ixy="0.0" ixz="0.0" iyy="0.001" iyz="0.0" izz="0.002"/>
-        </inertial>
-        <visual>
-            <origin xyz="0 0 0" rpy="1.5708 0 0"/>
-            <geometry>
-                <cylinder radius="${wheel_radius}" length="${wheel_width}"/>
-            </geometry>
-            <material name="black">
-                <color rgba="0 0 0 1"/>
-            </material>
-        </visual>
-            <collision>
-            <origin xyz="0 0 0" rpy="1.5708 0 0"/>
-            <geometry>
-                <cylinder radius="${wheel_radius}" length="${wheel_width}"/>
-            </geometry>
-        </collision>
+      <inertial>
+        <origin xyz="0 0 0"/>
+        <mass value="0.8"/>
+        <inertia ixx="0.001" ixy="0.0" ixz="0.0" iyy="0.001" iyz="0.0" izz="0.002"/>
+      </inertial>
+      <visual>
+        <origin xyz="0 0 0" rpy="1.5708 0 0"/>
+        <geometry>
+          <cylinder radius="${wheel_radius}" length="${wheel_width}"/>
+        </geometry>
+        <material name="black">
+          <color rgba="0 0 0 1"/>
+        </material>
+      </visual>
+      <collision>
+        <origin xyz="0 0 0" rpy="1.5708 0 0"/>
+        <geometry>
+          <cylinder radius="${wheel_radius}" length="${wheel_width}"/>
+        </geometry>
+      </collision>
     </link>
-  <joint name="${robot_name}/caster_joint_back" type="fixed">
-    <parent link="${robot_name}/base_link"/>
-    <child link="${robot_name}/caster_link_back"/>
-    <origin xyz="-${base_length/4} 0 0"/>
-  </joint>
-  <link name="${robot_name}/caster_link_back">
-    <visual>
-      <origin xyz="0 0 0"/>
-      <geometry>
-        <sphere radius="0.04"/>
-      </geometry>
-      <material name="black">
-        <color rgba="0 0 0 1"/>
-      </material>
-    </visual>
-    <collision>
-      <origin xyz="0 0 0" rpy="0 0 0"/>
-      <geometry>
-        <sphere radius="0.04"/>
-      </geometry>
-    </collision>
-  </link>
-  <joint name="${robot_name}/caster_joint_front" type="fixed">
-    <parent link="${robot_name}/base_link"/>
-    <child link="${robot_name}/caster_link_front"/>
-    <origin xyz="${base_length/4} 0 0"/>
-  </joint>
-  <link name="${robot_name}/caster_link_front">
-    <visual>
-      <origin xyz="0 0 0"/>
-      <geometry>
-        <sphere radius="0.04"/>
-      </geometry>
-      <material name="black">
-        <color rgba="0 0 0 1"/>
-      </material>
-    </visual>
-    <collision>
-      <origin xyz="0 0 0" rpy="0 0 0"/>
-      <geometry>
-        <sphere radius="0.04"/>
-      </geometry>
-    </collision>
-  </link>
-  <joint name="${robot_name}/laser_joint" type="fixed">
-    <parent link="${robot_name}/base_link"/>
-    <child link="${robot_name}/laser_link"/>
-    <origin xyz="${base_length/2-0.05} 0 ${base_height+0.03}" rpy="0 0 0"/>
-  </joint>
-  <link name="${robot_name}/laser_link">
-    <visual>
-      <origin xyz="0 0 0"/>
-      <geometry>
-        <cylinder radius="0.04" length="0.06"/>
-      </geometry>
-      <material name="purple">
-        <color rgba="0.1 0.01 0.8 1.0"/>
-      </material>
-    </visual>
-    <collision>
-      <origin xyz="0 0 0"/>
-      <geometry>
-        <cylinder radius="0.04" length="0.06"/>
-      </geometry>
-    </collision>
-  </link>
-  <joint name="${robot_name}/imu_joint" type="fixed">
-    <parent link="${robot_name}/base_link"/>
-    <child link="${robot_name}/imu_link"/>
-    <origin xyz="0 0 ${base_height/2}"/>
-  </joint>
-  <link name="${robot_name}/imu_link"/>
+    <joint name="${robot_name}/caster_joint_back" type="fixed">
+      <parent link="${robot_name}/base_link"/>
+      <child link="${robot_name}/caster_link_back"/>
+      <origin xyz="-${base_length/4} 0 0"/>
+    </joint>
+    <link name="${robot_name}/caster_link_back">
+      <visual>
+        <origin xyz="0 0 0"/>
+        <geometry>
+          <sphere radius="0.04"/>
+        </geometry>
+        <material name="black">
+          <color rgba="0 0 0 1"/>
+        </material>
+      </visual>
+      <collision>
+        <origin xyz="0 0 0" rpy="0 0 0"/>
+        <geometry>
+          <sphere radius="0.04"/>
+        </geometry>
+      </collision>
+    </link>
+    <joint name="${robot_name}/caster_joint_front" type="fixed">
+      <parent link="${robot_name}/base_link"/>
+      <child link="${robot_name}/caster_link_front"/>
+      <origin xyz="${base_length/4} 0 0"/>
+    </joint>
+    <link name="${robot_name}/caster_link_front">
+      <visual>
+        <origin xyz="0 0 0"/>
+        <geometry>
+          <sphere radius="0.04"/>
+        </geometry>
+        <material name="black">
+          <color rgba="0 0 0 1"/>
+        </material>
+      </visual>
+      <collision>
+        <origin xyz="0 0 0" rpy="0 0 0"/>
+        <geometry>
+          <sphere radius="0.04"/>
+        </geometry>
+      </collision>
+    </link>
+    <joint name="${robot_name}/laser_joint" type="fixed">
+      <parent link="${robot_name}/base_link"/>
+      <child link="${robot_name}/laser_link"/>
+      <origin xyz="${base_length/2-0.05} 0 ${base_height+0.03}" rpy="0 0 0"/>
+    </joint>
+    <link name="${robot_name}/laser_link">
+      <visual>
+        <origin xyz="0 0 0"/>
+        <geometry>
+          <cylinder radius="0.04" length="0.06"/>
+        </geometry>
+        <material name="purple">
+          <color rgba="0.1 0.01 0.8 1.0"/>
+        </material>
+      </visual>
+      <collision>
+        <origin xyz="0 0 0"/>
+        <geometry>
+          <cylinder radius="0.04" length="0.06"/>
+        </geometry>
+      </collision>
+    </link>
+    <joint name="${robot_name}/imu_joint" type="fixed">
+      <parent link="${robot_name}/base_link"/>
+      <child link="${robot_name}/imu_link"/>
+      <origin xyz="0 0 ${base_height/2}"/>
+    </joint>
+    <link name="${robot_name}/imu_link"/>
     <xacro:tug_gazebo robot_name="$(arg robot_name)"/>
   </xacro:macro>
