Commit message: added lidar
Signed-off-by: Tanishq Chaudhary <tanishqchaudhary101010@gmail.com>

File: robots_description/urdf/tug.gazebo.xacro (robot description, xacro)
@@ -62,6 +62,65 @@
 				<publish_wheel_tf>true</publish_wheel_tf>
 				<odometry_frame>world</odometry_frame>
-				<robot_base_frame>${robot_name}/base_link</robot_base_frame>
+				<robot_base_frame>${robot_name}/robot</robot_base_frame>
 			</plugin>
+		</gazebo>
+		<gazebo reference="${robot_name}/imu">
+			<gravity>true</gravity>
+			<sensor name="${robot_name}_imu_sensor" type="imu">
+				<always_on>true</always_on>
+				<update_rate>100</update_rate>
+				<visualize>false</visualize>
+				<plugin name="${robot_name}_imu_gazebo_plugin" filename="libgazebo_ros_imu_sensor.so">
+					<ros>
+						<namespace>${robot_name}</namespace>
+						<remapping>~/out:=imu</remapping>
+					</ros>
+					<bodyName>${robot_name}/imu</bodyName>
+					<updateRateHZ>10.0</updateRateHZ>
+					<xyzOffset>0 0 0</xyzOffset>
+					<rpyOffset>0 0 0</rpyOffset>
+					<frameName>${robot_name}/imu</frameName>
+					<initialOrientationAsReference>false</initialOrientationAsReference>
+				</plugin>
+				<pose>0 0 0 0 0 0</pose>
+			</sensor>
+		</gazebo>
+		<gazebo reference="${robot_name}/lidar">
+			<sensor name="${robot_name}_lidar" type="ray">
+				<always_on>true</always_on>
+				<update_rate>10</update_rate>				<!-- scan frequency in Hz -->
+				<visualize>true</visualize>
+				<!-- Laser ray configuration -->
+				<ray>
+					<scan>
+						<horizontal>
+							<samples>36</samples>							<!-- number of points per scan (low precision) -->
+							<resolution>1</resolution>
+							<min_angle>-1.57</min_angle>							<!-- -90 degrees -->
+							<max_angle>1.57</max_angle>							<!-- 90 degrees -->
+						</horizontal>
+					</scan>
+					<range>
+						<min>0.1</min>
+						<max>10.0</max>
+						<resolution>0.01</resolution>
+					</range>
+					<!-- Low-precision Gaussian noise -->
+					<noise type="gaussian">
+						<mean>0.0</mean>
+						<stddev>0.05</stddev>
+					</noise>
+				</ray>
+				<plugin name="${robot_name}_lidar_gazebo_plugin" filename="libgazebo_ros_ray_sensor.so">
+					<ros>
+						<namespace>${robot_name}</namespace>
+						<remapping>~/out:=lidar/points</remapping>
+					</ros>
+					<output_type>sensor_msgs/PointCloud2</output_type>
+					<min_intensity>100.0</min_intensity>
+					<frame_name>${robot_name}/lidar</frame_name>
+				</plugin>
+				<pose>0 0 0 0 0 0</pose>				<!-- adjust height above base_link -->
+			</sensor>
 		</gazebo>
 	</xacro:macro>

File: robots_description/urdf/tug.model.xacro (robot description, xacro)
@@ -12,5 +12,5 @@
     <xacro:property name="wheel_gap_from_base" value="0.01"/>
     <xacro:property name="wheel_separation" value="${base_width/2 + wheel_width/2 + wheel_gap_from_base}"/>
-    <link name="${robot_name}/base_link">
+    <link name="${robot_name}/robot">
       <inertial>
         <origin xyz="0 0 0" rpy="0 0 0"/>
@@ -35,5 +35,5 @@
     </link>
     <joint name="${robot_name}/joint_left_wheel" type="continuous">
-      <parent link="${robot_name}/base_link"/>
+      <parent link="${robot_name}/robot"/>
       <child link="${robot_name}/left_wheel"/>
       <origin xyz="0 ${wheel_separation} ${wheel_radius/2}" rpy="0 0 0"/>
@@ -63,5 +63,5 @@
     </link>
     <joint name="${robot_name}/joint_right_wheel" type="continuous">
-      <parent link="${robot_name}/base_link"/>
+      <parent link="${robot_name}/robot"/>
       <child link="${robot_name}/right_wheel"/>
       <origin xyz="0 -${wheel_separation} ${wheel_radius/2}" rpy="0 0 0"/>
@@ -91,5 +91,5 @@
     </link>
     <joint name="${robot_name}/caster_joint_back" type="fixed">
-      <parent link="${robot_name}/base_link"/>
+      <parent link="${robot_name}/robot"/>
       <child link="${robot_name}/caster_link_back"/>
       <origin xyz="-${base_length/4} 0 0"/>
@@ -113,5 +113,5 @@
     </link>
     <joint name="${robot_name}/caster_joint_front" type="fixed">
-      <parent link="${robot_name}/base_link"/>
+      <parent link="${robot_name}/robot"/>
       <child link="${robot_name}/caster_link_front"/>
       <origin xyz="${base_length/4} 0 0"/>
@@ -134,10 +134,10 @@
       </collision>
     </link>
-    <joint name="${robot_name}/laser_joint" type="fixed">
-      <parent link="${robot_name}/base_link"/>
-      <child link="${robot_name}/laser_link"/>
+    <joint name="${robot_name}/lidar_joint" type="fixed">
+      <parent link="${robot_name}/robot"/>
+      <child link="${robot_name}/lidar"/>
       <origin xyz="${base_length/2-0.05} 0 ${base_height+0.03}" rpy="0 0 0"/>
     </joint>
-    <link name="${robot_name}/laser_link">
+    <link name="${robot_name}/lidar">
       <visual>
         <origin xyz="0 0 0"/>
@@ -157,9 +157,9 @@
     </link>
     <joint name="${robot_name}/imu_joint" type="fixed">
-      <parent link="${robot_name}/base_link"/>
-      <child link="${robot_name}/imu_link"/>
+      <parent link="${robot_name}/robot"/>
+      <child link="${robot_name}/imu"/>
       <origin xyz="0 0 ${base_height/2}"/>
     </joint>
-    <link name="${robot_name}/imu_link"/>
+    <link name="${robot_name}/imu"/>
     <xacro:tug_gazebo robot_name="$(arg robot_name)"/>
   </xacro:macro>
