Commit message: depth cam frame
Signed-off-by: Tanishq Chaudhary <tanishqchaudhary101010@gmail.com>

File: robots_description/urdf/common.gazebo.xacro (robot description, xacro)
@@ -64,5 +64,5 @@
         <gazebo reference="${robot_name}/lidar">
             <material>Gazebo/Blue</material>
-            <sensor name="${robot_name}_lidar" type="ray">
+            <sensor name="lidar" type="ray">
                 <always_on>true</always_on>
                 <update_rate>10</update_rate>                <!-- scan frequency in Hz -->

File: robots_description/urdf/picker.gazebo.xacro (robot description, xacro)
@@ -11,5 +11,5 @@
 		<gazebo reference="${robot_name}/imu">
 			<gravity>true</gravity>
-			<sensor name="${robot_name}_imu_sensor" type="imu">
+			<sensor name="imu_sensor" type="imu">
 				<always_on>true</always_on>
 				<update_rate>100</update_rate>
@@ -30,4 +30,33 @@
 			</sensor>
 		</gazebo>
+		<!-- Depth Camera Sensor -->
+		<gazebo reference="${robot_name}/depth_camera_sensor">
+			<sensor name="depth_camera" type="depth">
+				<always_on>true</always_on>
+				<update_rate>30.0</update_rate>
+				<visualize>true</visualize>
+				<camera>
+					<horizontal_fov>1.047</horizontal_fov>					<!-- ~60 degrees -->
+					<image>
+						<width>640</width>
+						<height>480</height>
+						<format>R8G8B8</format>
+					</image>
+					<clip>
+						<near>0.05</near>
+						<far>5.0</far>
+					</clip>
+				</camera>
+				<!-- Gazebo ROS plugin -->
+				<plugin name="${robot_name}_depth_camera_gazebo_plugin" filename="libgazebo_ros_camera.so">
+					<ros>
+						<!-- Replace <robot_namespace> with your robot name or namespace -->
+						<namespace>${robot_name}</namespace>
+						<remapping>~/out:=depth</remapping>
+					</ros>
+					<frame_name>${robot_name}/depth_camera_sensor</frame_name>
+				</plugin>
+			</sensor>
+		</gazebo>
 	</xacro:macro>
 </robot>

File: robots_description/urdf/picker.model.xacro (robot description, xacro)
@@ -90,5 +90,19 @@
       </collision>
     </link>
-    <joint name="${robot_name}/caster_joint_back" type="fixed">
+    <joint name="${robot_name}/joint_depth_camera" type="fixed">
+      <parent link="${robot_name}/robot"/>
+      <child link="${robot_name}/depth_camera"/>
+      <origin xyz="${base_length/2} 0 0"/>
+    </joint>
+    <link name="${robot_name}/depth_camera">
+    </link>
+    <joint name="${robot_name}/joint_depth_camera_sensor" type="fixed">
+      <parent link="${robot_name}/depth_camera"/>
+      <child link="${robot_name}/depth_camera_sensor"/>
+      <origin xyz="0 0 0" rpy="0 0 0"/>
+    </joint>
+    <link name="${robot_name}/depth_camera_sensor">
+    </link>
+    <joint name="${robot_name}/joint_caster_back" type="fixed">
       <parent link="${robot_name}/robot"/>
       <child link="${robot_name}/caster_link_back"/>
@@ -112,5 +126,5 @@
       </collision>
     </link>
-    <joint name="${robot_name}/caster_joint_front" type="fixed">
+    <joint name="${robot_name}/joint_caster_front" type="fixed">
       <parent link="${robot_name}/robot"/>
       <child link="${robot_name}/caster_link_front"/>
