Commit message: added picker robot
Signed-off-by: Tanishq Chaudhary <tanishqchaudhary101010@gmail.com>

File: robots_description/urdf/picker.gazebo.xacro (robot description, xacro)
@@ -1,11 +1,11 @@
 <?xml version="1.0"?>
-<robot name="tug_gazebo"
+<robot name="picker_gazebo"
 	xmlns:xacro="http://ros.org/wiki/xacro">
-	<xacro:arg name="robot_name" default="tug_X"/>
+	<xacro:arg name="robot_name" default="picker_X"/>
 	<xacro:include filename="$(find robots_description)/urdf/common.gazebo.xacro"/>
-	<xacro:macro name="tug_gazebo" params="robot_name">
+	<xacro:macro name="picker_gazebo" params="robot_name">
 		<xacro:common_gazebo robot_name="$(arg robot_name)"/>
 		<gazebo reference="${robot_name}/robot">
-			<material>Gazebo/Red</material>
+			<material>Gazebo/Green</material>
 		</gazebo>
 		<gazebo reference="${robot_name}/imu">

Commit message: fix
Signed-off-by: Tanishq Chaudhary <tanishqchaudhary101010@gmail.com>

File: robots_description/urdf/picker.gazebo.xacro (robot description, xacro)
@@ -32,4 +32,5 @@
 		<!-- Depth Camera Sensor -->
 		<gazebo reference="${robot_name}/depth_camera_sensor">
+			<material>Gazebo/Black</material>
 			<sensor name="depth_camera" type="depth">
 				<always_on>true</always_on>

File: robots_description/urdf/picker.model.xacro (robot description, xacro)
@@ -93,7 +93,27 @@
       <parent link="${robot_name}/robot"/>
       <child link="${robot_name}/depth_camera"/>
-      <origin xyz="${base_length/2} 0 0"/>
+      <origin xyz="${base_length/2+0.0125} 0 ${base_height-0.0125}"/>
     </joint>
     <link name="${robot_name}/depth_camera">
+    <inertial>
+        <origin xyz="0 0 0" rpy="0 0 0"/>
+        <mass value="0.1"/>
+        <inertia ixx=".1" ixy="0.0" ixz="0.0" iyy=".12" iyz="0.0" izz=".12"/>
+      </inertial>
+      <visual>
+        <geometry>
+          <box size="0.025 0.075 0.025"/>
+        </geometry>
+        <origin xyz="0 0 0"/>
+        <material name="black">
+          <color rgba="0 0 0 1.0"/>
+        </material>
+      </visual>
+      <collision>
+        <geometry>
+          <box size="0.025 0.075 0.025"/>
+        </geometry>
+        <origin xyz="0 0 0"/>
+      </collision>
     </link>
     <joint name="${robot_name}/joint_depth_camera_sensor" type="fixed">
