Commit message: refactor pkg name
Signed-off-by: Tanishq Chaudhary <tanishqchaudhary101010@gmail.com>

File: multi-robot-navigation/urdf/common.gazebo.xacro (robot description, xacro)
@@ -2,7 +2,7 @@
 <robot name="common_gazebo"
     xmlns:xacro="http://ros.org/wiki/xacro">
-    <xacro:arg name="robot_name" default="picker_X"/>
-    <xacro:macro name="common_gazebo" params="robot_name">
-        <gazebo reference="${robot_name}/left_wheel">
+    <xacro:arg name="ns" default="picker_X"/>
+    <xacro:macro name="common_gazebo" params="ns">
+        <gazebo reference="${ns}/left_wheel">
             <mu1>1.0</mu1>
             <mu2>1.0</mu2>
@@ -13,5 +13,5 @@
             <material>Gazebo/Black</material>
         </gazebo>
-        <gazebo reference="${robot_name}/right_wheel">
+        <gazebo reference="${ns}/right_wheel">
             <mu1>1.0</mu1>
             <mu2>1.0</mu2>
@@ -22,5 +22,5 @@
             <material>Gazebo/Black</material>
         </gazebo>
-        <gazebo reference="${robot_name}/caster_link_back">
+        <gazebo reference="${ns}/caster_link_back">
             <mu1>0.0</mu1>
             <mu2>0.0</mu2>
@@ -31,5 +31,5 @@
             <material>Gazebo/Black</material>
         </gazebo>
-        <gazebo reference="${robot_name}/caster_link_front">
+        <gazebo reference="${ns}/caster_link_front">
             <mu1>0.0</mu1>
             <mu2>0.0</mu2>
@@ -41,11 +41,11 @@
         </gazebo>
         <gazebo>
-            <plugin name='${robot_name}_diff_drive_gazebo_plugin' filename='libgazebo_ros_diff_drive.so'>
+            <plugin name='${ns}_diff_drive_gazebo_plugin' filename='libgazebo_ros_diff_drive.so'>
                 <ros>
-                    <namespace>${robot_name}</namespace>
+                    <namespace>${ns}</namespace>
                 </ros>
                 <!-- wheels -->
-                <left_joint>${robot_name}/joint_left_wheel</left_joint>
-                <right_joint>${robot_name}/joint_right_wheel</right_joint>
+                <left_joint>${ns}/joint_left_wheel</left_joint>
+                <right_joint>${ns}/joint_right_wheel</right_joint>
                 <!-- kinematics -->
                 <wheel_separation>${wheel_separation}</wheel_separation>
@@ -58,9 +58,9 @@
                 <publish_odom_tf>true</publish_odom_tf>
                 <publish_wheel_tf>true</publish_wheel_tf>
-                <odometry_frame>${robot_name}/odom</odometry_frame>
-                <robot_base_frame>${robot_name}/robot</robot_base_frame>
+                <odometry_frame>${ns}/odom</odometry_frame>
+                <robot_base_frame>${ns}/robot</robot_base_frame>
             </plugin>
         </gazebo>
-        <gazebo reference="${robot_name}/lidar">
+        <gazebo reference="${ns}/lidar">
             <material>Gazebo/Blue</material>
             <sensor name="lidar" type="ray">
@@ -89,12 +89,12 @@
                     </noise>
                 </ray>
-                <plugin name="${robot_name}_lidar_gazebo_plugin" filename="libgazebo_ros_ray_sensor.so">
+                <plugin name="${ns}_lidar_gazebo_plugin" filename="libgazebo_ros_ray_sensor.so">
                     <ros>
-                        <namespace>${robot_name}</namespace>
+                        <namespace>${ns}</namespace>
                         <remapping>~/out:=lidar/points</remapping>
                     </ros>
                     <output_type>sensor_msgs/LaserScan</output_type>
                     <min_intensity>100.0</min_intensity>
-                    <frame_name>${robot_name}/lidar</frame_name>
+                    <frame_name>${ns}/lidar</frame_name>
                 </plugin>
                 <pose>0 0 0 0 0 0</pose>                <!-- adjust height above base_link -->

File: multi-robot-navigation/urdf/picker.gazebo.xacro (robot description, xacro)
@@ -2,12 +2,12 @@
 <robot name="picker_gazebo"
 	xmlns:xacro="http://ros.org/wiki/xacro">
-	<xacro:arg name="robot_name" default="picker_X"/>
-	<xacro:include filename="$(find robots_description)/urdf/common.gazebo.xacro"/>
-	<xacro:macro name="picker_gazebo" params="robot_name">
-		<xacro:common_gazebo robot_name="$(arg robot_name)"/>
-		<gazebo reference="${robot_name}/robot">
+	<xacro:arg name="ns" default="picker_X"/>
+	<xacro:include filename="$(find multi-robot-navigation)/urdf/common.gazebo.xacro"/>
+	<xacro:macro name="picker_gazebo" params="ns">
+		<xacro:common_gazebo ns="$(arg ns)"/>
+		<gazebo reference="${ns}/robot">
 			<material>Gazebo/Green</material>
 		</gazebo>
-		<gazebo reference="${robot_name}/imu">
+		<gazebo reference="${ns}/imu">
 			<gravity>true</gravity>
 			<sensor name="imu_sensor" type="imu">
@@ -15,14 +15,14 @@
 				<update_rate>100</update_rate>
 				<visualize>false</visualize>
-				<plugin name="${robot_name}_imu_gazebo_plugin" filename="libgazebo_ros_imu_sensor.so">
+				<plugin name="${ns}_imu_gazebo_plugin" filename="libgazebo_ros_imu_sensor.so">
 					<ros>
-						<namespace>${robot_name}</namespace>
+						<namespace>${ns}</namespace>
 						<remapping>~/out:=imu</remapping>
 					</ros>
-					<bodyName>${robot_name}/imu</bodyName>
+					<bodyName>${ns}/imu</bodyName>
 					<updateRateHZ>10.0</updateRateHZ>
 					<xyzOffset>0 0 0</xyzOffset>
 					<rpyOffset>0 0 0</rpyOffset>
-					<frameName>${robot_name}/imu</frameName>
+					<frameName>${ns}/imu</frameName>
 					<initialOrientationAsReference>false</initialOrientationAsReference>
 				</plugin>
@@ -30,7 +30,9 @@
 			</sensor>
 		</gazebo>
+		<gazebo reference="${ns}/depth_camera">
+			<material>Gazebo/Black</material>
+		</gazebo>
 		<!-- Depth Camera Sensor -->
-		<gazebo reference="${robot_name}/depth_camera_sensor">
-			<material>Gazebo/Black</material>
+		<gazebo reference="${ns}/depth_camera_sensor">
 			<sensor name="depth_camera" type="depth">
 				<always_on>true</always_on>
@@ -50,11 +52,11 @@
 				</camera>
 				<!-- Gazebo ROS plugin -->
-				<plugin name="${robot_name}_depth_camera_gazebo_plugin" filename="libgazebo_ros_camera.so">
+				<plugin name="${ns}_depth_camera_gazebo_plugin" filename="libgazebo_ros_camera.so">
 					<ros>
 						<!-- Replace <robot_namespace> with your robot name or namespace -->
-						<namespace>${robot_name}</namespace>
+						<namespace>${ns}</namespace>
 						<remapping>~/out:=depth</remapping>
 					</ros>
-					<frame_name>${robot_name}/depth_camera_sensor</frame_name>
+					<frame_name>${ns}/depth_camera_sensor</frame_name>
 				</plugin>
 			</sensor>

File: multi-robot-navigation/urdf/picker.model.xacro (robot description, xacro)
@@ -1,8 +1,8 @@
 <?xml version="1.0"?>
-<robot name="tug"
+<robot name="picker"
   xmlns:xacro="http://www.ros.org/wiki/xacro">
-  <xacro:arg name="robot_name" default="tug_X"/>
-  <xacro:include filename="$(find robots_description)/urdf/tug.gazebo.xacro"/>
-  <xacro:macro name="tug_model" params="robot_name">
+  <xacro:arg name="ns" default="picker_X"/>
+  <xacro:include filename="$(find multi-robot-navigation)/urdf/picker.gazebo.xacro"/>
+  <xacro:macro name="picker_model" params="ns">
     <xacro:property name="base_length" value="0.6"/>
     <xacro:property name="base_width" value="0.45"/>
@@ -12,5 +12,5 @@
     <xacro:property name="wheel_gap_from_base" value="0.01"/>
     <xacro:property name="wheel_separation" value="${base_width/2 + wheel_width/2 + wheel_gap_from_base}"/>
-    <link name="${robot_name}/robot">
+    <link name="${ns}/robot">
       <inertial>
         <origin xyz="0 0 0" rpy="0 0 0"/>
@@ -23,6 +23,6 @@
         </geometry>
         <origin xyz="0 0 ${base_height/2}"/>
-        <material name="red">
-          <color rgba="1 0 0.01 1.0"/>
+        <material name="green">
+          <color rgba="0.01 1 0 1.0"/>
         </material>
       </visual>
@@ -34,11 +34,11 @@
       </collision>
     </link>
-    <joint name="${robot_name}/joint_left_wheel" type="continuous">
-      <parent link="${robot_name}/robot"/>
-      <child link="${robot_name}/left_wheel"/>
+    <joint name="${ns}/joint_left_wheel" type="continuous">
+      <parent link="${ns}/robot"/>
+      <child link="${ns}/left_wheel"/>
       <origin xyz="0 ${wheel_separation} ${wheel_radius/2}" rpy="0 0 0"/>
       <axis xyz="0 1 0"/>
     </joint>
-    <link name="${robot_name}/left_wheel">
+    <link name="${ns}/left_wheel">
       <inertial>
         <origin xyz="0 0 0"/>
@@ -62,11 +62,11 @@
       </collision>
     </link>
-    <joint name="${robot_name}/joint_right_wheel" type="continuous">
-      <parent link="${robot_name}/robot"/>
-      <child link="${robot_name}/right_wheel"/>
+    <joint name="${ns}/joint_right_wheel" type="continuous">
+      <parent link="${ns}/robot"/>
+      <child link="${ns}/right_wheel"/>
       <origin xyz="0 -${wheel_separation} ${wheel_radius/2}" rpy="0 0 0"/>
       <axis xyz="0 1 0"/>
     </joint>
-    <link name="${robot_name}/right_wheel">
+    <link name="${ns}/right_wheel">
       <inertial>
         <origin xyz="0 0 0"/>
@@ -90,54 +90,88 @@
       </collision>
     </link>
-    <joint name="${robot_name}/caster_joint_back" type="fixed">
-      <parent link="${robot_name}/robot"/>
-      <child link="${robot_name}/caster_link_back"/>
+    <joint name="${ns}/joint_depth_camera" type="fixed">
+      <parent link="${ns}/robot"/>
+      <child link="${ns}/depth_camera"/>
+      <origin xyz="${base_length/2+0.0125} 0 ${base_height-0.0125}"/>
+    </joint>
+    <link name="${ns}/depth_camera">
+    <inertial>
+        <origin xyz="0 0 0" rpy="0 0 0"/>
+        <mass value="0.1"/>
+        <inertia ixx=".1" ixy="0.0" ixz="0.0" iyy=".12" iyz="0.0" izz=".12"/>
+      </inertial>
+      <visual>
+        <geometry>
+          <box size="0.025 0.075 0.025"/>
+        </geometry>
+        <origin xyz="0 0 0"/>
+        <material name="black">
+          <color rgba="0 0 0 1.0"/>
+        </material>
+      </visual>
+      <collision>
+        <geometry>
+          <box size="0.025 0.075 0.025"/>
+        </geometry>
+        <origin xyz="0 0 0"/>
+      </collision>
+    </link>
+    <joint name="${ns}/joint_depth_camera_sensor" type="fixed">
+      <parent link="${ns}/depth_camera"/>
+      <child link="${ns}/depth_camera_sensor"/>
+      <origin xyz="0 0 0" rpy="0 0 0"/>
+    </joint>
+    <link name="${ns}/depth_camera_sensor">
+    </link>
+    <joint name="${ns}/joint_caster_back" type="fixed">
+      <parent link="${ns}/robot"/>
+      <child link="${ns}/caster_link_back"/>
       <origin xyz="-${base_length/4} 0 0"/>
     </joint>
-    <link name="${robot_name}/caster_link_back">
-      <visual>
-        <origin xyz="0 0 0"/>
-        <geometry>
-          <sphere radius="0.04"/>
-        </geometry>
-        <material name="black">
-          <color rgba="0 0 0 1"/>
-        </material>
-      </visual>
-      <collision>
-        <origin xyz="0 0 0" rpy="0 0 0"/>
-        <geometry>
-          <sphere radius="0.04"/>
-        </geometry>
-      </collision>
-    </link>
-    <joint name="${robot_name}/caster_joint_front" type="fixed">
-      <parent link="${robot_name}/robot"/>
-      <child link="${robot_name}/caster_link_front"/>
+    <link name="${ns}/caster_link_back">
+      <visual>
+        <origin xyz="0 0 0"/>
+        <geometry>
+          <sphere radius="0.04"/>
+        </geometry>
+        <material name="black">
+          <color rgba="0 0 0 1"/>
+        </material>
+      </visual>
+      <collision>
+        <origin xyz="0 0 0" rpy="0 0 0"/>
+        <geometry>
+          <sphere radius="0.04"/>
+        </geometry>
+      </collision>
+    </link>
+    <joint name="${ns}/joint_caster_front" type="fixed">
+      <parent link="${ns}/robot"/>
+      <child link="${ns}/caster_link_front"/>
       <origin xyz="${base_length/4} 0 0"/>
     </joint>
-    <link name="${robot_name}/caster_link_front">
-      <visual>
-        <origin xyz="0 0 0"/>
-        <geometry>
-          <sphere radius="0.04"/>
-        </geometry>
-        <material name="black">
-          <color rgba="0 0 0 1"/>
-        </material>
-      </visual>
-      <collision>
-        <origin xyz="0 0 0" rpy="0 0 0"/>
-        <geometry>
-          <sphere radius="0.04"/>
-        </geometry>
-      </collision>
-    </link>
-    <joint name="${robot_name}/lidar_joint" type="fixed">
-      <parent link="${robot_name}/robot"/>
-      <child link="${robot_name}/lidar"/>
+    <link name="${ns}/caster_link_front">
+      <visual>
+        <origin xyz="0 0 0"/>
+        <geometry>
+          <sphere radius="0.04"/>
+        </geometry>
+        <material name="black">
+          <color rgba="0 0 0 1"/>
+        </material>
+      </visual>
+      <collision>
+        <origin xyz="0 0 0" rpy="0 0 0"/>
+        <geometry>
+          <sphere radius="0.04"/>
+        </geometry>
+      </collision>
+    </link>
+    <joint name="${ns}/lidar_joint" type="fixed">
+      <parent link="${ns}/robot"/>
+      <child link="${ns}/lidar"/>
       <origin xyz="${base_length/2-0.05} 0 ${base_height+0.03}" rpy="0 0 0"/>
     </joint>
-    <link name="${robot_name}/lidar">
+    <link name="${ns}/lidar">
       <visual>
         <origin xyz="0 0 0"/>
@@ -156,11 +190,11 @@
       </collision>
     </link>
-    <joint name="${robot_name}/imu_joint" type="fixed">
-      <parent link="${robot_name}/robot"/>
-      <child link="${robot_name}/imu"/>
+    <joint name="${ns}/imu_joint" type="fixed">
+      <parent link="${ns}/robot"/>
+      <child link="${ns}/imu"/>
       <origin xyz="0 0 ${base_height/2}"/>
     </joint>
-    <link name="${robot_name}/imu"/>
-    <xacro:tug_gazebo robot_name="$(arg robot_name)"/>
+    <link name="${ns}/imu"/>
+    <xacro:picker_gazebo ns="$(arg ns)"/>
   </xacro:macro>
 </robot>

File: multi-robot-navigation/urdf/tug.gazebo.xacro (robot description, xacro)
@@ -2,27 +2,27 @@
 <robot name="tug_gazebo"
 	xmlns:xacro="http://ros.org/wiki/xacro">
-	<xacro:arg name="robot_name" default="tug_X"/>
-	<xacro:include filename="$(find robots_description)/urdf/common.gazebo.xacro"/>
-	<xacro:macro name="tug_gazebo" params="robot_name">
-		<xacro:common_gazebo robot_name="$(arg robot_name)"/>
-		<gazebo reference="${robot_name}/robot">
+	<xacro:arg name="ns" default="tug_X"/>
+	<xacro:include filename="$(find multi-robot-navigation)/urdf/common.gazebo.xacro"/>
+	<xacro:macro name="tug_gazebo" params="ns">
+		<xacro:common_gazebo ns="$(arg ns)"/>
+		<gazebo reference="${ns}/robot">
 			<material>Gazebo/Red</material>
 		</gazebo>
-		<gazebo reference="${robot_name}/imu">
+		<gazebo reference="${ns}/imu">
 			<gravity>true</gravity>
-			<sensor name="${robot_name}_imu_sensor" type="imu">
+			<sensor name="${ns}_imu_sensor" type="imu">
 				<always_on>true</always_on>
 				<update_rate>100</update_rate>
 				<visualize>false</visualize>
-				<plugin name="${robot_name}_imu_gazebo_plugin" filename="libgazebo_ros_imu_sensor.so">
+				<plugin name="${ns}_imu_gazebo_plugin" filename="libgazebo_ros_imu_sensor.so">
 					<ros>
-						<namespace>${robot_name}</namespace>
+						<namespace>${ns}</namespace>
 						<remapping>~/out:=imu</remapping>
 					</ros>
-					<bodyName>${robot_name}/imu</bodyName>
+					<bodyName>${ns}/imu</bodyName>
 					<updateRateHZ>10.0</updateRateHZ>
 					<xyzOffset>0 0 0</xyzOffset>
 					<rpyOffset>0 0 0</rpyOffset>
-					<frameName>${robot_name}/imu</frameName>
+					<frameName>${ns}/imu</frameName>
 					<initialOrientationAsReference>false</initialOrientationAsReference>
 				</plugin>

File: multi-robot-navigation/urdf/tug.model.xacro (robot description, xacro)
@@ -1,8 +1,8 @@
 <?xml version="1.0"?>
-<robot name="picker"
+<robot name="tug"
   xmlns:xacro="http://www.ros.org/wiki/xacro">
-  <xacro:arg name="robot_name" default="picker_X"/>
-  <xacro:include filename="$(find robots_description)/urdf/picker.gazebo.xacro"/>
-  <xacro:macro name="picker_model" params="robot_name">
+  <xacro:arg name="ns" default="tug_X"/>
+  <xacro:include filename="$(find multi-robot-navigation)/urdf/tug.gazebo.xacro"/>
+  <xacro:macro name="tug_model" params="ns">
     <xacro:property name="base_length" value="0.6"/>
     <xacro:property name="base_width" value="0.45"/>
@@ -12,5 +12,5 @@
     <xacro:property name="wheel_gap_from_base" value="0.01"/>
     <xacro:property name="wheel_separation" value="${base_width/2 + wheel_width/2 + wheel_gap_from_base}"/>
-    <link name="${robot_name}/robot">
+    <link name="${ns}/robot">
       <inertial>
         <origin xyz="0 0 0" rpy="0 0 0"/>
@@ -23,6 +23,6 @@
         </geometry>
         <origin xyz="0 0 ${base_height/2}"/>
-        <material name="green">
-          <color rgba="0.01 1 0 1.0"/>
+        <material name="red">
+          <color rgba="1 0 0.01 1.0"/>
         </material>
       </visual>
@@ -34,11 +34,11 @@
       </collision>
     </link>
-    <joint name="${robot_name}/joint_left_wheel" type="continuous">
-      <parent link="${robot_name}/robot"/>
-      <child link="${robot_name}/left_wheel"/>
+    <joint name="${ns}/joint_left_wheel" type="continuous">
+      <parent link="${ns}/robot"/>
+      <child link="${ns}/left_wheel"/>
       <origin xyz="0 ${wheel_separation} ${wheel_radius/2}" rpy="0 0 0"/>
       <axis xyz="0 1 0"/>
     </joint>
-    <link name="${robot_name}/left_wheel">
+    <link name="${ns}/left_wheel">
       <inertial>
         <origin xyz="0 0 0"/>
@@ -62,11 +62,11 @@
       </collision>
     </link>
-    <joint name="${robot_name}/joint_right_wheel" type="continuous">
-      <parent link="${robot_name}/robot"/>
-      <child link="${robot_name}/right_wheel"/>
+    <joint name="${ns}/joint_right_wheel" type="continuous">
+      <parent link="${ns}/robot"/>
+      <child link="${ns}/right_wheel"/>
       <origin xyz="0 -${wheel_separation} ${wheel_radius/2}" rpy="0 0 0"/>
       <axis xyz="0 1 0"/>
     </joint>
-    <link name="${robot_name}/right_wheel">
+    <link name="${ns}/right_wheel">
       <inertial>
         <origin xyz="0 0 0"/>
@@ -90,44 +90,10 @@
       </collision>
     </link>
-    <joint name="${robot_name}/joint_depth_camera" type="fixed">
-      <parent link="${robot_name}/robot"/>
-      <child link="${robot_name}/depth_camera"/>
-      <origin xyz="${base_length/2+0.0125} 0 ${base_height-0.0125}"/>
-    </joint>
-    <link name="${robot_name}/depth_camera">
-    <inertial>
-        <origin xyz="0 0 0" rpy="0 0 0"/>
-        <mass value="0.1"/>
-        <inertia ixx=".1" ixy="0.0" ixz="0.0" iyy=".12" iyz="0.0" izz=".12"/>
-      </inertial>
-      <visual>
-        <geometry>
-          <box size="0.025 0.075 0.025"/>
-        </geometry>
-        <origin xyz="0 0 0"/>
-        <material name="black">
-          <color rgba="0 0 0 1.0"/>
-        </material>
-      </visual>
-      <collision>
-        <geometry>
-          <box size="0.025 0.075 0.025"/>
-        </geometry>
-        <origin xyz="0 0 0"/>
-      </collision>
-    </link>
-    <joint name="${robot_name}/joint_depth_camera_sensor" type="fixed">
-      <parent link="${robot_name}/depth_camera"/>
-      <child link="${robot_name}/depth_camera_sensor"/>
-      <origin xyz="0 0 0" rpy="0 0 0"/>
-    </joint>
-    <link name="${robot_name}/depth_camera_sensor">
-    </link>
-    <joint name="${robot_name}/joint_caster_back" type="fixed">
-      <parent link="${robot_name}/robot"/>
-      <child link="${robot_name}/caster_link_back"/>
+    <joint name="${ns}/caster_joint_back" type="fixed">
+      <parent link="${ns}/robot"/>
+      <child link="${ns}/caster_link_back"/>
       <origin xyz="-${base_length/4} 0 0"/>
     </joint>
-    <link name="${robot_name}/caster_link_back">
+    <link name="${ns}/caster_link_back">
       <visual>
         <origin xyz="0 0 0"/>
@@ -146,10 +112,10 @@
       </collision>
     </link>
-    <joint name="${robot_name}/joint_caster_front" type="fixed">
-      <parent link="${robot_name}/robot"/>
-      <child link="${robot_name}/caster_link_front"/>
+    <joint name="${ns}/caster_joint_front" type="fixed">
+      <parent link="${ns}/robot"/>
+      <child link="${ns}/caster_link_front"/>
       <origin xyz="${base_length/4} 0 0"/>
     </joint>
-    <link name="${robot_name}/caster_link_front">
+    <link name="${ns}/caster_link_front">
       <visual>
         <origin xyz="0 0 0"/>
@@ -168,10 +134,10 @@
       </collision>
     </link>
-    <joint name="${robot_name}/lidar_joint" type="fixed">
-      <parent link="${robot_name}/robot"/>
-      <child link="${robot_name}/lidar"/>
+    <joint name="${ns}/lidar_joint" type="fixed">
+      <parent link="${ns}/robot"/>
+      <child link="${ns}/lidar"/>
       <origin xyz="${base_length/2-0.05} 0 ${base_height+0.03}" rpy="0 0 0"/>
     </joint>
-    <link name="${robot_name}/lidar">
+    <link name="${ns}/lidar">
       <visual>
         <origin xyz="0 0 0"/>
@@ -190,11 +156,11 @@
       </collision>
     </link>
-    <joint name="${robot_name}/imu_joint" type="fixed">
-      <parent link="${robot_name}/robot"/>
-      <child link="${robot_name}/imu"/>
+    <joint name="${ns}/imu_joint" type="fixed">
+      <parent link="${ns}/robot"/>
+      <child link="${ns}/imu"/>
       <origin xyz="0 0 ${base_height/2}"/>
     </joint>
-    <link name="${robot_name}/imu"/>
-    <xacro:picker_gazebo robot_name="$(arg robot_name)"/>
+    <link name="${ns}/imu"/>
+    <xacro:tug_gazebo ns="$(arg ns)"/>
   </xacro:macro>
 </robot>
